Commit message: Update my_robot.xacro

File: my_robot/urdf/my_robot.xacro (robot description, xacro)
@@ -179,11 +179,11 @@
   </joint>
 <gazebo reference="left_wheel">
-    <material>Gazebo/Green</material>
+    <material>Gazebo/Blue</material>
 </gazebo>
 <gazebo reference="right_wheel">
-    <material>Gazebo/Green</material>
+    <material>Gazebo/Blue</material>
 </gazebo>
 <gazebo reference="chassis">
-    <material>Gazebo/Blue</material>
+    <material>Gazebo/Green</material>
 </gazebo>
 <gazebo reference="camera">
